File: sensie.brd (EAGLE design)
At the start: 38.1 x 25.4 mm, 25 parts, among them J2 BATT, Q1 MOSFET-PCHANNELSMD, Q2 MOSFET-NCHANNELBSS138, Q3 20MHz

Commit message: Sent to OshPark.
Parts:
- added POW!: (no value), SparkFun-LED:LED-0603
- added R2, R3, R4: (no value), SparkFun-Passives:0603-RES
- moved Q2 0.13 mm to (10.2, 12.1), turned to 270 degrees
Connections:
- new net N$3: POW!.A, R2.1
- net 3.3V: now also R3.2, R4.2
- net AN0: now also R4.1
- net COUNTER: now also R3.1
- net GND: now also POW!.C
- net VIN_USB: now also R2.2
Routing:
- net 3.3V: track 95.1 -> 110.9 mm
- net GND: track 149.5 -> 139.4 mm, vias 2 -> 3
- net COUNTER: track 16.6 -> 19.3 mm
- net VIN_USB: track 17.7 -> 20.1 mm, vias 1 -> 2
- net AN0: track 9.48 -> 11.8 mm
- net ANALOG_ENABLE: track 9.75 -> 7.63 mm
- net N$3: track 0.00 -> 1.29 mm
Other:
- board text added: "(rev.1)"
- board text added: "1-wire bus pullups"
- board text added: "AN0"
- board text added: "AN1"
- board text added: "AN11"
- board text added: "AN2"
- board text added: "AN3"
- board text added: "AN9"
- board text added: "Analog Inputs"
- board text added: "BATTERY 4.5V - 15V"
- board text added: "Counter"
- board text added: "MAGIC"
- board text added: "Sensie"
- board text added: "by bitlab. 2013"
- board text removed: "bitlab. 2013"
