File: sensie.sch (EAGLE design)
At the start: 28 parts, among them J2 BATT, Q1 MOSFET-PCHANNELSMD, Q2 MOSFET-NCHANNELBSS138, Q3 20MHz

Commit message: About to refactor headers.
Parts:
- renumbered LED2 to PWR
Connections:
- net ANALOG_VPP_ENABLE renamed ANALOG_ENABLE
- removed net N$6: 3.3V.1, 3.3V.2, 3.3V.3, 3.3V.4, 3.3V.5, 3.3V.6, 3.3V.7, Q2.S
- net 3.3V: now also 3.3V.1, 3.3V.2, 3.3V.3, 3.3V.4, 3.3V.5, 3.3V.6, 3.3V.7
- net GND: now also Q2.S
Other:
- moved on the sheet: 3.3V, GND, Q2
Changed lines of the file:
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@@
 <part name="GND1" library="SparkFun" deviceset="GND" device=""/>
 <part name="R3" library="SparkFun" deviceset="RESISTOR" device="" value="330"/>
-<part name="LED2" library="SparkFun" deviceset="LED" device="0603"/>
+<part name="PWR" library="SparkFun" deviceset="LED" device="0603"/>
 <part name="GND4" library="SparkFun" deviceset="GND" device=""/>
 <part name="C1" library="SparkFun" deviceset="CAP" device="0805" value="0.1uF"/>
@@
 <part name="GND11" library="supply1" deviceset="GND" device=""/>
 <part name="Q2" library="SparkFun-DiscreteSemi" deviceset="MOSFET-NCHANNEL" device="BSS138"/>
+<part name="GND12" library="supply1" deviceset="GND" device=""/>
 </parts>
 <sheets>
@@
 <instance part="SENSOR" gate="G$1" x="279.4" y="83.82" rot="R180"/>
 <instance part="BLUETOOTH" gate="G$1" x="279.4" y="63.5" rot="R180"/>
-<instance part="3.3V" gate="G$1" x="330.2" y="45.72"/>
+<instance part="3.3V" gate="G$1" x="327.66" y="63.5"/>
 <instance part="SENSE" gate="G$1" x="279.4" y="43.18" rot="R180"/>
-<instance part="GND" gate="G$1" x="304.8" y="45.72"/>
+<instance part="GND" gate="G$1" x="353.06" y="63.5"/>
 <instance part="GND6" gate="1" x="336.55" y="198.12"/>
 <instance part="R5" gate="G$1" x="302.26" y="203.2" rot="R90"/>
@@
 <instance part="GND1" gate="1" x="101.6" y="144.78"/>
 <instance part="R3" gate="G$1" x="213.36" y="50.8" rot="R270"/>
-<instance part="LED2" gate="G$1" x="213.36" y="43.18"/>
+<instance part="PWR" gate="G$1" x="213.36" y="43.18"/>
 <instance part="GND4" gate="1" x="213.36" y="35.56"/>
 <instance part="C1" gate="G$1" x="101.6" y="149.86"/>
@@
 <instance part="GND9" gate="1" x="177.546" y="147.32"/>
 <instance part="JP1" gate="G$1" x="182.626" y="153.67"/>
-<instance part="GND11" gate="1" x="309.88" y="35.56"/>
-<instance part="Q2" gate="G$1" x="335.28" y="68.58"/>
+<instance part="GND11" gate="1" x="358.14" y="53.34"/>
+<instance part="Q2" gate="G$1" x="332.74" y="45.72"/>
+<instance part="GND12" gate="1" x="332.74" y="35.56"/>
 </instances>
 <busses>
@@
 </segment>
 <segment>
-<pinref part="LED2" gate="G$1" pin="C"/>
+<pinref part="PWR" gate="G$1" pin="C"/>
 <pinref part="GND4" gate="1" pin="GND"/>
 </segment>
@@
 <pinref part="GND" gate="G$1" pin="7"/>
 <pinref part="GND" gate="G$1" pin="6"/>
-<wire x1="309.88" y1="55.88" x2="309.88" y2="53.34" width="0.1524" layer="91"/>
+<wire x1="358.14" y1="73.66" x2="358.14" y2="71.12" width="0.1524" layer="91"/>
 <pinref part="GND" gate="G$1" pin="5"/>
-<wire x1="309.88" y1="50.8" x2="309.88" y2="53.34" width="0.1524" layer="91"/>
+<wire x1="358.14" y1="68.58" x2="358.14" y2="71.12" width="0.1524" layer="91"/>
 <pinref part="GND" gate="G$1" pin="4"/>
-<wire x1="309.88" y1="48.26" x2="309.88" y2="50.8" width="0.1524" layer="91"/>
+<wire x1="358.14" y1="66.04" x2="358.14" y2="68.58" width="0.1524" layer="91"/>
 <pinref part="GND" gate="G$1" pin="3"/>
-<wire x1="309.88" y1="45.72" x2="309.88" y2="48.26" width="0.1524" layer="91"/>
+<wire x1="358.14" y1="63.5" x2="358.14" y2="66.04" width="0.1524" layer="91"/>
 <pinref part="GND" gate="G$1" pin="2"/>
-<wire x1="309.88" y1="43.18" x2="309.88" y2="45.72" width="0.1524" layer="91"/>
+<wire x1="358.14" y1="60.96" x2="358.14" y2="63.5" width="0.1524" layer="91"/>
 <pinref part="GND" gate="G$1" pin="1"/>
-<wire x1="309.88" y1="40.64" x2="309.88" y2="43.18" width="0.1524" layer="91"/>
+<wire x1="358.14" y1="58.42" x2="358.14" y2="60.96" width="0.1524" layer="91"/>
 <pinref part="GND11" gate="1" pin="GND"/>
-<wire x1="309.88" y1="40.64" x2="309.88" y2="38.1" width="0.1524" layer="91"/>
+<wire x1="358.14" y1="58.42" x2="358.14" y2="55.88" width="0.1524" layer="91"/>
+</segment>
+<segment>
+<pinref part="Q2" gate="G$1" pin="S"/>
+<pinref part="GND12" gate="1" pin="GND"/>
+<wire x1="332.74" y1="40.64" x2="332.74" y2="38.1" width="0.1524" layer="91"/>
 </segment>
 </net>
@@
 <segment>
 <pinref part="R3" gate="G$1" pin="2"/>
-<pinref part="LED2" gate="G$1" pin="A"/>
+<pinref part="PWR" gate="G$1" pin="A"/>
 </segment>
 </net>
@@
 </segment>
 <segment>
+<pinref part="3.3V" gate="G$1" pin="7"/>
+<pinref part="3.3V" gate="G$1" pin="6"/>
+<wire x1="332.74" y1="73.66" x2="332.74" y2="71.12" width="0.1524" layer="91"/>
+<pinref part="3.3V" gate="G$1" pin="5"/>
+<wire x1="332.74" y1="71.12" x2="332.74" y2="68.58" width="0.1524" layer="91"/>
+<pinref part="3.3V" gate="G$1" pin="4"/>
+<wire x1="332.74" y1="68.58" x2="332.74" y2="66.04" width="0.1524" layer="91"/>
+<pinref part="3.3V" gate="G$1" pin="3"/>
+<wire x1="332.74" y1="66.04" x2="332.74" y2="63.5" width="0.1524" layer="91"/>
+<pinref part="3.3V" gate="G$1" pin="2"/>
+<wire x1="332.74" y1="63.5" x2="332.74" y2="60.96" width="0.1524" layer="91"/>
+<pinref part="3.3V" gate="G$1" pin="1"/>
+<wire x1="332.74" y1="60.96" x2="332.74" y2="58.42" width="0.1524" layer="91"/>
+<wire x1="332.74" y1="73.66" x2="332.74" y2="81.28" width="0.1524" layer="91"/>
+<label x="332.74" y="81.28" size="1.778" layer="95"/>
 <pinref part="Q2" gate="G$1" pin="D"/>
-<wire x1="335.28" y1="73.66" x2="335.28" y2="78.74" width="0.1524" layer="91"/>
-<label x="335.28" y="78.74" size="1.778" layer="95"/>
+<wire x1="332.74" y1="58.42" x2="332.74" y2="50.8" width="0.1524" layer="91"/>
 </segment>
 </net>
@@
 </segment>
 </net>
-<net name="ANALOG_VPP_ENABLE" class="0">
+<net name="ANALOG_ENABLE" class="0">
 <segment>
 <wire x1="143.51" y1="191.77" x2="161.29" y2="191.77" width="0.1524" layer="91"/>
@@
 <segment>
 <pinref part="Q2" gate="G$1" pin="G"/>
-<wire x1="327.66" y1="68.58" x2="320.04" y2="68.58" width="0.1524" layer="91"/>
-<label x="302.26" y="68.58" size="1.778" layer="95"/>
+<wire x1="325.12" y1="45.72" x2="317.5" y2="45.72" width="0.1524" layer="91"/>
+<label x="306.832" y="45.72" size="1.778" layer="95"/>
 </segment>
 </net>
@@
 </segment>
 </net>
-<net name="N$6" class="0">
-<segment>
-<pinref part="Q2" gate="G$1" pin="S"/>
-<pinref part="3.3V" gate="G$1" pin="7"/>
-<wire x1="335.28" y1="63.5" x2="335.28" y2="55.88" width="0.1524" layer="91"/>
-<pinref part="3.3V" gate="G$1" pin="6"/>
-<wire x1="335.28" y1="55.88" x2="335.28" y2="53.34" width="0.1524" layer="91"/>
-<pinref part="3.3V" gate="G$1" pin="5"/>
-<wire x1="335.28" y1="53.34" x2="335.28" y2="50.8" width="0.1524" layer="91"/>
-<pinref part="3.3V" gate="G$1" pin="4"/>
-<wire x1="335.28" y1="50.8" x2="335.28" y2="48.26" width="0.1524" layer="91"/>
-<pinref part="3.3V" gate="G$1" pin="3"/>
-<wire x1="335.28" y1="48.26" x2="335.28" y2="45.72" width="0.1524" layer="91"/>
-<pinref part="3.3V" gate="G$1" pin="2"/>
-<wire x1="335.28" y1="45.72" x2="335.28" y2="43.18" width="0.1524" layer="91"/>
-<pinref part="3.3V" gate="G$1" pin="1"/>
-<wire x1="335.28" y1="43.18" x2="335.28" y2="40.64" width="0.1524" layer="91"/>
-</segment>
-</net>

Commit message: About to refactor uC.
Parts:
- removed SENSE: (no value), SparkFun-Connectors:M07
- added JP2: (no value), SparkFun-Connectors:M07
Connections:
- removed net AN6: SENSE.7
- new net COUNTER: JP2.1, U$3.RA4/AN4
- net AN0: now also JP2.2; no longer SENSE.1
- net AN1: now also JP2.3; no longer SENSE.2
- net AN2: now also JP2.4; no longer SENSE.3
- net AN3: now also JP2.5; no longer SENSE.4
- net AN4: now also JP2.6; no longer SENSE.5
- net AN5: now also JP2.7; no longer SENSE.6
Changed lines of the file:
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@@
 <part name="BLUETOOTH" library="SparkFun-Connectors" deviceset="M04" device="PTH"/>
 <part name="3.3V" library="SparkFun-Connectors" deviceset="M07" device=""/>
-<part name="SENSE" library="SparkFun-Connectors" deviceset="M07" device=""/>
 <part name="GND" library="SparkFun-Connectors" deviceset="M07" device=""/>
 <part name="GND6" library="SparkFun" deviceset="GND" device=""/>
@@
 <part name="Q2" library="SparkFun-DiscreteSemi" deviceset="MOSFET-NCHANNEL" device="BSS138"/>
 <part name="GND12" library="supply1" deviceset="GND" device=""/>
+<part name="JP2" library="SparkFun-Connectors" deviceset="M07" device=""/>
 </parts>
 <sheets>
@@
 <instance part="BLUETOOTH" gate="G$1" x="279.4" y="63.5" rot="R180"/>
 <instance part="3.3V" gate="G$1" x="327.66" y="63.5"/>
-<instance part="SENSE" gate="G$1" x="279.4" y="43.18" rot="R180"/>
 <instance part="GND" gate="G$1" x="353.06" y="63.5"/>
 <instance part="GND6" gate="1" x="336.55" y="198.12"/>
@@
 <instance part="Q2" gate="G$1" x="332.74" y="45.72"/>
 <instance part="GND12" gate="1" x="332.74" y="35.56"/>
+<instance part="JP2" gate="G$1" x="279.4" y="38.1" rot="R180"/>
 </instances>
 <busses>
@@
 </segment>
 <segment>
-<pinref part="SENSE" gate="G$1" pin="1"/>
-<wire x1="274.32" y1="48.26" x2="264.16" y2="48.26" width="0.1524" layer="91"/>
-<label x="264.16" y="48.26" size="1.778" layer="95"/>
+<wire x1="274.32" y1="40.64" x2="264.16" y2="40.64" width="0.1524" layer="91"/>
+<label x="264.16" y="40.64" size="1.778" layer="95"/>
+<pinref part="JP2" gate="G$1" pin="2"/>
 </segment>
 </net>
@@
 </segment>
 <segment>
-<pinref part="SENSE" gate="G$1" pin="2"/>
-<wire x1="274.32" y1="45.72" x2="264.16" y2="45.72" width="0.1524" layer="91"/>
-<label x="264.16" y="45.72" size="1.778" layer="95"/>
+<wire x1="274.32" y1="38.1" x2="264.16" y2="38.1" width="0.1524" layer="91"/>
+<label x="264.16" y="38.1" size="1.778" layer="95"/>
+<pinref part="JP2" gate="G$1" pin="3"/>
 </segment>
 </net>
@@
 </segment>
 <segment>
-<pinref part="SENSE" gate="G$1" pin="3"/>
-<wire x1="274.32" y1="43.18" x2="264.16" y2="43.18" width="0.1524" layer="91"/>
-<label x="264.16" y="43.18" size="1.778" layer="95"/>
+<wire x1="274.32" y1="35.56" x2="264.16" y2="35.56" width="0.1524" layer="91"/>
+<label x="264.16" y="35.56" size="1.778" layer="95"/>
+<pinref part="JP2" gate="G$1" pin="4"/>
 </segment>
 </net>
@@
 </segment>
 <segment>
-<pinref part="SENSE" gate="G$1" pin="4"/>
-<wire x1="274.32" y1="40.64" x2="264.16" y2="40.64" width="0.1524" layer="91"/>
-<label x="264.16" y="40.64" size="1.778" layer="95"/>
+<wire x1="274.32" y1="33.02" x2="264.16" y2="33.02" width="0.1524" layer="91"/>
+<label x="264.16" y="33.02" size="1.778" layer="95"/>
+<pinref part="JP2" gate="G$1" pin="5"/>
 </segment>
 </net>
@@
 </segment>
 <segment>
-<pinref part="SENSE" gate="G$1" pin="5"/>
-<wire x1="274.32" y1="38.1" x2="264.16" y2="38.1" width="0.1524" layer="91"/>
-<label x="264.16" y="38.1" size="1.778" layer="95"/>
+<wire x1="274.32" y1="30.48" x2="264.16" y2="30.48" width="0.1524" layer="91"/>
+<label x="264.16" y="30.48" size="1.778" layer="95"/>
+<pinref part="JP2" gate="G$1" pin="6"/>
 </segment>
 </net>
@@
 </segment>
 <segment>
-<pinref part="SENSE" gate="G$1" pin="6"/>
-<wire x1="274.32" y1="35.56" x2="264.16" y2="35.56" width="0.1524" layer="91"/>
-<label x="264.16" y="35.56" size="1.778" layer="95"/>
-</segment>
-</net>
-<net name="AN6" class="0">
-<segment>
-<pinref part="SENSE" gate="G$1" pin="7"/>
-<wire x1="274.32" y1="33.02" x2="264.16" y2="33.02" width="0.1524" layer="91"/>
-<label x="264.16" y="33.02" size="1.778" layer="95"/>
+<wire x1="274.32" y1="27.94" x2="264.16" y2="27.94" width="0.1524" layer="91"/>
+<label x="264.16" y="27.94" size="1.778" layer="95"/>
+<pinref part="JP2" gate="G$1" pin="7"/>
 </segment>
 </net>
@@
 </segment>
 </net>
+<net name="COUNTER" class="0">
+<segment>
+<pinref part="JP2" gate="G$1" pin="1"/>
+<wire x1="274.32" y1="43.18" x2="263.906" y2="43.18" width="0.1524" layer="91"/>
+<label x="264.16" y="43.18" size="1.778" layer="95"/>
+</segment>
+<segment>
+<pinref part="U$3" gate="G$1" pin="RA4/AN4"/>
+<wire x1="105.41" y1="179.07" x2="88.9" y2="179.07" width="0.1524" layer="91"/>
+<label x="89.916" y="179.07" size="1.778" layer="95"/>
+</segment>
+</net>

Commit message: Routing cleanup.
Parts:
- removed PWR: (no value), SparkFun:LED0603
- removed R3: 330, SparkFun:RESISTOR
Connections:
- removed net N$7: PWR.A, R3.2
- net 3.3V: now also SENSOR.1; no longer SENSOR.6
- net GND: now also SENSOR.6, U$2.1; no longer PWR.C, SENSOR.1
Changed lines of the file:
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@@
 <part name="U$3" library="SparkFun" deviceset="PIC18F2455" device="SMD"/>
 <part name="GND1" library="SparkFun" deviceset="GND" device=""/>
-<part name="R3" library="SparkFun" deviceset="RESISTOR" device="" value="330"/>
-<part name="PWR" library="SparkFun" deviceset="LED" device="0603"/>
-<part name="GND4" library="SparkFun" deviceset="GND" device=""/>
 <part name="C1" library="SparkFun" deviceset="CAP" device="0805" value="0.1uF"/>
 <part name="GND5" library="SparkFun" deviceset="GND" device=""/>
@@
 <instance part="U$3" gate="G$1" x="125.73" y="173.99"/>
 <instance part="GND1" gate="1" x="101.6" y="144.78"/>
-<instance part="R3" gate="G$1" x="213.36" y="50.8" rot="R270"/>
-<instance part="PWR" gate="G$1" x="213.36" y="43.18"/>
-<instance part="GND4" gate="1" x="213.36" y="35.56"/>
 <instance part="C1" gate="G$1" x="101.6" y="149.86"/>
 <instance part="GND5" gate="1" x="351.79" y="198.12"/>
@@
 </segment>
 <segment>
-<pinref part="PWR" gate="G$1" pin="C"/>
-<pinref part="GND4" gate="1" pin="GND"/>
-</segment>
-<segment>
 <pinref part="GND1" gate="1" pin="GND"/>
 <pinref part="C1" gate="G$1" pin="2"/>
@@
 </segment>
 <segment>
-<pinref part="GND3" gate="1" pin="GND"/>
-<wire x1="312.42" y1="106.68" x2="312.42" y2="104.14" width="0.1524" layer="91"/>
-<wire x1="312.42" y1="104.14" x2="315.214" y2="104.14" width="0.1524" layer="91"/>
-</segment>
-<segment>
 <pinref part="BLUETOOTH" gate="G$1" pin="2"/>
 <wire x1="274.32" y1="63.5" x2="264.16" y2="63.5" width="0.1524" layer="91"/>
 <label x="264.16" y="63.5" size="1.778" layer="95"/>
-</segment>
-<segment>
-<pinref part="SENSOR" gate="G$1" pin="1"/>
-<wire x1="274.32" y1="88.9" x2="264.16" y2="88.9" width="0.1524" layer="91"/>
-<label x="264.16" y="88.9" size="1.778" layer="95"/>
 </segment>
 <segment>
@@
 <wire x1="332.74" y1="40.64" x2="332.74" y2="38.1" width="0.1524" layer="91"/>
 </segment>
+<segment>
+<pinref part="GND3" gate="1" pin="GND"/>
+<pinref part="U$2" gate="G$1" pin="1"/>
+<wire x1="312.42" y1="106.68" x2="312.42" y2="104.14" width="0.1524" layer="91"/>
+<wire x1="312.42" y1="104.14" x2="314.96" y2="104.14" width="0.1524" layer="91"/>
+</segment>
+<segment>
+<pinref part="SENSOR" gate="G$1" pin="6"/>
+<wire x1="274.32" y1="76.2" x2="264.16" y2="76.2" width="0.1524" layer="91"/>
+<label x="264.16" y="76.2" size="1.778" layer="95"/>
+</segment>
 </net>
 <net name="VIN_USB" class="0">
@@
 </segment>
 </net>
-<net name="N$7" class="0">
-<segment>
-<pinref part="R3" gate="G$1" pin="2"/>
-<pinref part="PWR" gate="G$1" pin="A"/>
-</segment>
-</net>
 <net name="3.3V" class="0">
 <segment>
@@
 <label x="264.16" y="66.04" size="1.778" layer="95"/>
 <label x="264.16" y="66.04" size="1.778" layer="95"/>
-</segment>
-<segment>
-<pinref part="SENSOR" gate="G$1" pin="6"/>
-<wire x1="274.32" y1="76.2" x2="264.16" y2="76.2" width="0.1524" layer="91"/>
-<label x="264.16" y="76.2" size="1.778" layer="95"/>
 </segment>
 <segment>
@@
 <wire x1="332.74" y1="58.42" x2="332.74" y2="50.8" width="0.1524" layer="91"/>
 </segment>
-</net>
+<segment>
+<pinref part="SENSOR" gate="G$1" pin="1"/>
+<wire x1="274.32" y1="88.9" x2="264.16" y2="88.9" width="0.1524" layer="91"/>
+<label x="264.16" y="88.9" size="1.778" layer="95"/>
+</segment>
+</net>
